File: VCAT/Dev/Project/STM32 Bluetooth.kicad_sch (KiCad schematic)
At the start: 41 parts, among them J1 USB_C_Receptacle_USB2.0_16P, J2 Conn_ARM_SWD_TagConnect_TC2030, J3 Conn_01x04, J4 Conn_Coaxial, SW1 SW_Push, U1 MIC5365-3.3YD5, U2 USBLC6-2SC6, U3 STM32WB55CEUx, Y1 32Khz768, Y2 32Mhz

Commit message: new schematic
Parts:
- removed J2: Conn_ARM_SWD_TagConnect_TC2030, Connector:Tag-Connect_TC2030-IDC-FP_2x03_P1.27mm_Vertical, symbol Connector:Conn_ARM_SWD_TagConnect_TC2030
- removed J3: Conn_01x04, Connector_Molex:Molex_Pico-EZmate_78171-0003_1x03-1MP_P1.20mm_Vertical, symbol Connector_Generic:Conn_01x04
- removed Y1: 32Khz768, Crystal:Crystal_SMD_2012-2Pin_2.0x1.2mm, symbol Device:Crystal
- removed Y2: 32Mhz, Crystal:Crystal_SMD_2016-4Pin_2.0x1.6mm, symbol Device:Crystal_GND24
- added J2: Conn_01x04, Connector_Molex:Molex_PicoBlade_53048-0410_1x04_P1.25mm_Horizontal, symbol Connector_Generic:Conn_01x04
- added J3: TC2030, Connector:Tag-Connect_TC2030-IDC-FP_2x03_P1.27mm_Vertical, symbol Connector:Conn_ARM_SWD_TagConnect_TC2030
- added X1: 32kHz768, Crystal:Crystal_SMD_2012-2Pin_2.0x1.2mm, symbol Device:Crystal
- added X2: 32MHz, Crystal:Crystal_SMD_2016-4Pin_2.0x1.6mm, symbol Device:Crystal_GND24
- C1, C16, C3: value 100n -> 4u7; footprint Capacitor_SMD:C_0402_1005Metric -> Capacitor_SMD:C_0603_1608Metric
- C13: value C -> 100n
- C14: value 100n -> 10p
- C15: value C -> 10p
- C17: value 100n -> 0p8
- C18: value 0p8 -> 0p3
- C19: value 0p3 -> 100n
- FLT1: footprint layout:DLF162500LT-5028A1 -> Library:DLF162500LT-5028A1
- J1: value USB_C_Receptacle_USB2.0_16P -> USB_C_Receptacle_USB2.0; footprint Connector_USB:USB_C_Receptacle_Amphenol_12401948E412A -> Connector_USB:USB_C_Receptacle_GCT_USB4105-xx-A_16P_TopMnt_Horizontal
- L3: value 10u -> 2n7; footprint Inductor_SMD:L_0805_2012Metric -> Inductor_SMD:L_0402_1005Metric
- SW1: footprint Button_Switch_SMD:SW_Push_SPST_NO_Alps_SKRK -> Button_Switch_SMD:SW_SPST_CK_RS282G05A3
- U1: footprint Package_TO_SOT_SMD:TSOT-23-5 -> Package_TO_SOT_SMD:SOT-23-5
- U3: value STM32WB55CEUx -> STM32WB55CEU
Connections:
- net BOOT0: now also C19.1; no longer C17.1
- net GND: now also J1.S1 (SHIELD), R1.2, R2.2, J2.4 (Pin_4), J3.5 (GND), X2.2, X2.4; no longer J1.SH (SHIELD), R1.1, R2.1
- net RF: now also C17.1; no longer C18.1
- net SMPSLX: no longer L1.2, L2.1
- net at J1.A5 (CC1): now also R2.1; no longer R2.2
- net at J1.B5 (CC2): now also R1.1; no longer R1.2
- net RF_ANT: now reaches FLT1.3 (OUT), J4.1 (In)
- net RF_MATCH: now reaches FLT1.1 (IN), L3.2
- net RF_MATCH: now also C18.1; no longer C19.1
- net USB_D-: now reaches U2.6 (I/O1), U3.37 (PA11)
- net LSE_OUT: now reaches C14.1
- net LSE_OUT: now also U3.3 (PC15), X1.1; no longer U3.7 (NRST)
- net UART_TXC: now reaches R4.1
- net UART_TXC: now also J2.2 (Pin_2)
- net UART_RXC: now reaches R5.1
- net UART_RXC: now also J2.3 (Pin_3)
- net +3.3V renamed +3V3
- net +3V3: now also J2.1 (Pin_1), J3.1 (VCC)
- net HSE_in renamed HCE_IN
- net HCE_IN: now also X2.3
- net HSE_out renamed HCE_OUT
- net HCE_OUT: now also X2.1
- net LEDA: no longer names the net of D1.2 (A), U3.16 (PA7)
- net LEDC: no longer names the net of D1.1 (K), R3.2
- net LSE_in renamed LSE_IN
- net LSE_IN: now also X1.2
- net LSE_out renamed SWD_NRST
- net SWD_NRST: now also U3.7 (NRST), J3.3 (~{RESET}); no longer U3.3 (PC15)
- net SVD_CLK renamed SWD_CLK
- net SWD_CLK: now also J3.4 (SWCLK)
- net SVD_DIO renamed SWD_DIO
- net SWD_DIO: now also J3.2 (SWDIO)
- net SVD_TRC renamed SWD_TRC
- net SWD_TRC: now also J3.6 (SWO)
- new net SMPSLXL: L1.2, L2.1
- no-connect marks 21 -> 22
Other:
- note added: "+5V To 3.3V LDO REGULATOR"
- note added: "BOOT0 Switch"
- note added: "Tag-Connect SWD Header"
- note added: "USB-C Connector"
- note removed: "SWD_NRST"
- title: (none) -> STM32 Bluetooth Hardware Design

Commit message: 1.5
Connections:
- net GND: no longer J4.2 (Ext)
- net RF_ANT: no longer J4.1 (In)
Other:
- moved on the sheet: J4
Changed lines of the file:
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@@
 	(symbol
 		(lib_id "Connector:Conn_Coaxial")
-		(at 269.24 106.68 0)
+		(at 270.51 104.14 0)
 		(unit 1)
 		(body_style 1)
@@
 		(fields_autoplaced yes)
 		(property "Reference" "J4"
-			(at 273.05 105.7032 0)
+			(at 274.32 103.1632 0)
 			(show_name no)
 			(do_not_autoplace no)
@@
 		)
 		(property "Value" "Conn_Coaxial"
-			(at 273.05 108.2432 0)
+			(at 274.32 105.7032 0)
 			(show_name no)
 			(do_not_autoplace no)
@@
 		)
 		(property "Footprint" "Connector_Coaxial:U.FL_Hirose_U.FL-R-SMT-1_Vertical"
-			(at 269.24 106.68 0)
+			(at 270.51 104.14 0)
 			(hide yes)
 			(show_name no)
@@
 		)
 		(property "Datasheet" "~"
-			(at 269.24 106.68 0)
+			(at 270.51 104.14 0)
 			(hide yes)
 			(show_name no)
@@
 		)
 		(property "Description" ""
-			(at 269.24 106.68 0)
+			(at 270.51 104.14 0)
 			(show_name no)
 			(do_not_autoplace no)
