File: VCAT/Ishan/Starter Project/Starter Project.kicad_sch (KiCad schematic)
At the start: 0 parts

Commit message: Added starter project KiCAD files and footprints
Parts:
- added C1, C10, C2, C3, C4, C5, C6, C9: 100n, Package_DFN_QFN:QFN-48-1EP_7x7mm_P0.5mm_EP5.6x5.6mm, symbol Device:C
- added C11, C7, C8: 4.7u, Package_DFN_QFN:QFN-48-1EP_7x7mm_P0.5mm_EP5.6x5.6mm, symbol Device:C
- added C12, C13: C, Package_DFN_QFN:QFN-48-1EP_7x7mm_P0.5mm_EP5.6x5.6mm, symbol Device:C
- added C14: 0.8p, Package_DFN_QFN:QFN-48-1EP_7x7mm_P0.5mm_EP5.6x5.6mm, symbol Device:C
- added C15: 0.3p, Package_DFN_QFN:QFN-48-1EP_7x7mm_P0.5mm_EP5.6x5.6mm, symbol Device:C
- added L1: 10n, Relay_THT:Relay_DPDT_Finder_30.22, symbol Device:L
- added L2: 10u, Relay_THT:Relay_DPDT_Finder_30.22, symbol Device:L
- added L3: 2.7n, symbol Device:L
- added U1: STM32WB55CEU6, Package_DFN_QFN:QFN-48-1EP_7x7mm_P0.5mm_EP5.6x5.6mm, symbol MCU_ST_STM32WB:STM32WB55CEUx
- added X1: 32.768kHz, symbol Device:Crystal
- added X2: 32mHz, Package_DFN_QFN:QFN-48-1EP_7x7mm_P0.5mm_EP5.6x5.6mm, symbol Device:Crystal_GND24
Connections:
- new net: C13.1, U1.2 (PC14), X1.2
- new net: C12.1, U1.3 (PC15), X1.1
- new net: C14.1, L3.1, U1.21 (RF1)
- new net: C15.1, L3.2
- new net +3.3V: C1.1, C10.1, C2.1, C3.1, C4.1, C5.1, C6.1, C7.1, C8.1, C9.1, U1.1 (VBAT), U1.20 (VDD), U1.23 (VDDRF), U1.34 (VDDSMPS), U1.35 (VDD), U1.40 (VDDUSB), U1.48 (VDD), U1.8 (VDDA)
- new net GND: C1.2, C10.2, C11.2, C12.2, C13.2, C14.2, C15.2, C2.2, C3.2, C4.2, C5.2, C6.2, C7.2, C8.2, C9.2, U1.22 (VSSRF), U1.32 (VSSSMPS), U1.49 (VSS), X2.2 (G), X2.4 (G)
- new net HSE_IN: U1.25 (OSC_IN), X2.3
- new net HSE_OUT: U1.24 (OSC_OUT), X2.1
- new net SMPSFB: C11.1, L2.2, U1.31 (VFBSMPS)
- new net SMPSLX: L1.1, U1.33 (VLXSMPS)
- new net SMPSLXL: L1.2, L2.1

Commit message: Schematic Done
Parts:
- added C1, C2: 4.7u, Capacitor_SMD:C_0603_1608Metric, symbol Device:C
- added C13, C19: 100n, Capacitor_SMD:C_0402_1005Metric, symbol Device:C
- added D1: LED, LED_SMD:LED_0402_1005Metric, symbol Device:LED
- added FLT1: DLF162500LT-5028A1, starterProjectLibraryFootprints:Untitled, symbol starterProjectLibrary:DLF162500LT-5028A1
- added J1: USB_C_Receptacle_USB2.0_16P, Connector_USB:USB_C_Receptacle_GCT_USB4105-xx-A_16P_TopMnt_Horizontal, symbol Connector:USB_C_Receptacle_USB2.0_16P
- added J2: Conn_01x04, Connector_Molex:Molex_PicoBlade_53048-0410_1x04_P1.25mm_Horizontal, symbol Connector_Generic:Conn_01x04
- added J3: TC2030, Connector:Tag-Connect_TC2030-IDC-FP_2x03_P1.27mm_Vertical, symbol Connector:Conn_ARM_SWD_TagConnect_TC2030
- added J4: Conn_Coaxial, Connector_Coaxial:U.FL_Hirose_U.FL-R-SMT-1_Vertical, symbol Connector:Conn_Coaxial
- added R1, R2, R6: 5.1K, Resistor_SMD:R_0402_1005Metric, symbol Device:R
- added R3, R4, R5, R7: 220R, Resistor_SMD:R_0402_1005Metric, symbol Device:R
- added SW1: SW_Push, Button_Switch_SMD:SW_SPST_CK_RS282G05A3, symbol Switch:SW_Push
- added U1: MIC5365-3.3YD5, Package_TO_SOT_SMD:TSOT-23-5, symbol Regulator_Linear:MIC5365-3.3YD5
- added U2: USBLC6-2SC6, Package_TO_SOT_SMD:SOT-23-6, symbol Power_Protection:USBLC6-2SC6
- C10: renamed from C8; footprint Package_DFN_QFN:QFN-48-1EP_7x7mm_P0.5mm_EP5.6x5.6mm -> Capacitor_SMD:C_0603_1608Metric
- C11: renamed from C9; footprint Package_DFN_QFN:QFN-48-1EP_7x7mm_P0.5mm_EP5.6x5.6mm -> Capacitor_SMD:C_0402_1005Metric
- C12: renamed from C10; footprint Package_DFN_QFN:QFN-48-1EP_7x7mm_P0.5mm_EP5.6x5.6mm -> Capacitor_SMD:C_0402_1005Metric
- C14: renamed from C11; footprint Package_DFN_QFN:QFN-48-1EP_7x7mm_P0.5mm_EP5.6x5.6mm -> Capacitor_SMD:C_0603_1608Metric
- C15: renamed from C14; footprint Package_DFN_QFN:QFN-48-1EP_7x7mm_P0.5mm_EP5.6x5.6mm -> Capacitor_SMD:C_0402_1005Metric
- C16: renamed from C15; footprint Package_DFN_QFN:QFN-48-1EP_7x7mm_P0.5mm_EP5.6x5.6mm -> Capacitor_SMD:C_0402_1005Metric
- C17: renamed from C12; value C -> 10p; footprint Package_DFN_QFN:QFN-48-1EP_7x7mm_P0.5mm_EP5.6x5.6mm -> Capacitor_SMD:C_0402_1005Metric
- C18: renamed from C13; value C -> 10p; footprint Package_DFN_QFN:QFN-48-1EP_7x7mm_P0.5mm_EP5.6x5.6mm -> Capacitor_SMD:C_0402_1005Metric
- C3: renamed from C7; footprint Package_DFN_QFN:QFN-48-1EP_7x7mm_P0.5mm_EP5.6x5.6mm -> Capacitor_SMD:C_0603_1608Metric
- C4: renamed from C1; footprint Package_DFN_QFN:QFN-48-1EP_7x7mm_P0.5mm_EP5.6x5.6mm -> Capacitor_SMD:C_0402_1005Metric
- C5: renamed from C2; footprint Package_DFN_QFN:QFN-48-1EP_7x7mm_P0.5mm_EP5.6x5.6mm -> Capacitor_SMD:C_0402_1005Metric
- C6: renamed from C3; footprint Package_DFN_QFN:QFN-48-1EP_7x7mm_P0.5mm_EP5.6x5.6mm -> Capacitor_SMD:C_0402_1005Metric
- C7: renamed from C4; footprint Package_DFN_QFN:QFN-48-1EP_7x7mm_P0.5mm_EP5.6x5.6mm -> Capacitor_SMD:C_0402_1005Metric
- C8: renamed from C5; footprint Package_DFN_QFN:QFN-48-1EP_7x7mm_P0.5mm_EP5.6x5.6mm -> Capacitor_SMD:C_0402_1005Metric
- C9: renamed from C6; footprint Package_DFN_QFN:QFN-48-1EP_7x7mm_P0.5mm_EP5.6x5.6mm -> Capacitor_SMD:C_0402_1005Metric
- L1: footprint Relay_THT:Relay_DPDT_Finder_30.22 -> Inductor_SMD:L_0402_1005Metric
- L2: footprint Relay_THT:Relay_DPDT_Finder_30.22 -> Inductor_SMD:L_0805_2012Metric
- L3: footprint (none) -> Inductor_SMD:L_0402_1005Metric
- X1: footprint (none) -> Crystal:Crystal_SMD_2012-2Pin_2.0x1.2mm
- X2: footprint Package_DFN_QFN:QFN-48-1EP_7x7mm_P0.5mm_EP5.6x5.6mm -> Crystal:Crystal_SMD_2016-4Pin_2.0x1.6mm
- renumbered U1 to U3
Connections:
- net +3.3V: now also C2.1, J2.4 (Pin_4), J3.1 (VCC), SW1.2, U1.5 (VOUT)
- net GND: now also C1.2, C13.2, C19.2, C2.2, FLT1.2 (GND), FLT1.4 (GND), J1.A1 (GND), J1.A12 (GND), J1.B1 (GND), J1.B12 (GND), J1.SH (SHIELD), J2.1 (Pin_1), J3.5 (GND), J4.2 (Ext), R1.2, R2.2, R5.1, R6.2, U1.2 (GND), U2.2 (GND)
- net LSE_IN: now reaches C18.1, U3.2 (PC14), X1.2
- net LSE_OUT: now reaches C17.1, U3.3 (PC15), X1.1
- net RF: now reaches C15.1, L3.1, U3.21 (RF1)
- net RF_MATCH: now reaches C16.1, L3.2
- net RF_MATCH: now also FLT1.1 (IN)
- net UART_TX: now reaches U3.11 (PA2)
- net UART_TX: now also R3.2
- net UART_RX: now reaches U3.12 (PA3)
- net UART_RX: now also R4.2
- net LED_A: now reaches U3.16 (PA7)
- net LED_A: now also D1.2 (A)
- net USB_D-: now reaches U3.37 (PA11)
- net USB_D-: now also J1.A7 (D-), J1.B7 (D-), U2.1 (I/O1), U2.6 (I/O1)
- net USB_D+: now reaches U3.38 (PA12)
- net USB_D+: now also J1.A6 (D+), J1.B6 (D+), U2.3 (I/O2), U2.4 (I/O2)
- net SWD_DIO: now reaches U3.39 (PA13)
- net SWD_DIO: now also J3.2 (SWDIO)
- net at U3.4 (PH3): now also C19.1, R6.1, R7.1
- net SWD_CLK: now reaches U3.41 (PA14)
- net SWD_CLK: now also J3.4 (SWCLK)
- net SWD_TRC: now reaches U3.43 (PB3)
- net SWD_TRC: now also J3.6 (SWO)
- net SWD_NRST: now reaches U3.7 (NRST)
- net SWD_NRST: now also C13.1, J3.3 (~{RESET})
- new net: R7.2, SW1.1
- new net +5V: C1.1, J1.A4 (VBUS), J1.A9 (VBUS), J1.B4 (VBUS), J1.B9 (VBUS), U1.1 (VIN), U1.3 (EN), U2.5 (VBUS)
- new net LED_K: D1.1 (K), R5.2
- new net RF_ANT: FLT1.3 (OUT), J4.1 (In)
- new net UART_RXC: J2.2 (Pin_2), R4.1
- new net UART_TXC: J2.3 (Pin_3), R3.1
- new net USB_CC1: J1.A5 (CC1), R2.1
- new net USB_CC2: J1.B5 (CC2), R1.1
- no-connect marks 0 -> 21
Other:
- note added: "(3.3-1.8)/220 = 7mA"
- note added: "+5V to +3.3V LDO Regulator"
- note added: "BOOT0 Switch"
- note added: "LSE (32.768kHz) & HSE (32MHz) Crystals"
- note added: "RF Front-End & u.FL Connector"
- note added: "STM32WB KiCAD STARTER PROJECT"
- note added: "STM32WB55 MCU"
- note added: "Tag-Connect SWD Header"
- note added: "UART HEADER"
- note added: "USB-Connector"
