File: PSYS/Tamoghna/Starter_proj/Starter_proj.kicad_pcb (KiCad board)
At the start: 4 copper layers, 0 parts

Commit message: AHHHHHHHH ALL MY NETS WERE FUCKED FIXED IT
Parts:
- added C1: 100n, Capacitor_SMD:C_0603_1608Metric, F.Cu at (92.5, 58.3)
- added C10: 4u7, Capacitor_SMD:C_0805_2012Metric, F.Cu at (104.8, 75.1)
- added C11: 10p, Capacitor_SMD:C_0402_1005Metric, F.Cu at (118.8, 58.0)
- added C12: 10p, Capacitor_SMD:C_0402_1005Metric, F.Cu at (118.8, 60.0)
- added C13: 0p8, Capacitor_SMD:C_0402_1005Metric, F.Cu at (118.8, 61.9)
- added C14: 0p3, Capacitor_SMD:C_0402_1005Metric, F.Cu at (118.8, 63.9)
- added C15: 100n, Capacitor_SMD:C_0603_1608Metric, F.Cu at (96.5, 60.8)
- added C16: 100n, Capacitor_SMD:C_0603_1608Metric, F.Cu at (96.5, 63.3)
- added C17: 100n, Capacitor_SMD:C_0603_1608Metric, F.Cu at (96.5, 65.8)
- added C18: 4u7, Capacitor_SMD:C_0805_2012Metric, F.Cu at (104.8, 78.1)
- added C19: 4u7, Capacitor_SMD:C_0805_2012Metric, F.Cu at (104.8, 81.1)
- added C2: 100n, Capacitor_SMD:C_0603_1608Metric, F.Cu at (92.5, 60.8)
- added C3: 100n, Capacitor_SMD:C_0603_1608Metric, F.Cu at (92.5, 63.3)
- added C4: 100n, Capacitor_SMD:C_0603_1608Metric, F.Cu at (92.5, 65.8)
- added C5: 4u7, Capacitor_SMD:C_0805_2012Metric, F.Cu at (104.8, 69.1)
- added C6: 100n, Capacitor_SMD:C_0603_1608Metric, F.Cu at (92.5, 68.3)
- added C7: 4u7, Capacitor_SMD:C_0805_2012Metric, F.Cu at (104.8, 72.1)
- added C8: 100n, Capacitor_SMD:C_0603_1608Metric, F.Cu at (92.5, 70.8)
- added C9: 100n, Capacitor_SMD:C_0603_1608Metric, F.Cu at (96.5, 58.3)
- added D1: LED, LED_SMD:LED_0603_1608Metric, F.Cu at (109.0, 87.7)
- added FLT1: DLF162500LT-5028A1, footprintlib:Untitled, F.Cu at (112.7, 87.5)
- added J1: Conn_Coaxial, Connector_Coaxial:U.FL_Hirose_U.FL-R-SMT-1_Vertical, F.Cu at (93.6, 85.1)
- added J2: Conn_ARM_SWD_TagConnect_TC2030, Connector:Tag-Connect_TC2030-IDC-FP_2x03_P1.27mm_Vertical, F.Cu at (111.8, 81.6)
- added J3: USB_C_Receptacle_USB2.0_16P, Connector_USB:USB_C_Receptacle_GCT_USB4105-xx-A_16P_TopMnt_Horizontal, F.Cu at (96.3, 77.3)
- added J4: Conn_01x04, Connector_Molex:Molex_PicoBlade_53047-0410_1x04_P1.25mm_Vertical, F.Cu at (118.0, 80.5)
- added L1: 10n, Inductor_SMD:L_0402_1005Metric, F.Cu at (118.1, 71.3)
- added L2: 10u, Inductor_SMD:L_0805_2012Metric, F.Cu at (118.9, 68.9)
- added L3: 2n7, Inductor_SMD:L_0402_1005Metric, F.Cu at (118.1, 73.3)
- added R1: 5k1, Resistor_SMD:R_0603_1608Metric, F.Cu at (96.5, 68.3)
- added R2: 220R, Resistor_SMD:R_0603_1608Metric, F.Cu at (96.5, 70.8)
- added R3: 5K1, Resistor_SMD:R_0603_1608Metric, F.Cu at (100.5, 58.3)
- added R4: 5K1, Resistor_SMD:R_0603_1608Metric, F.Cu at (100.5, 60.8)
- added R5: 220R, Resistor_SMD:R_0603_1608Metric, F.Cu at (100.5, 63.3)
- added R6: 220R, Resistor_SMD:R_0603_1608Metric, F.Cu at (100.5, 65.8)
- added R7: 220R, Resistor_SMD:R_0603_1608Metric, F.Cu at (100.5, 68.3)
- added SW2: SW_SPDT, footprintlib:SW_Wurth_WS-SLSV_450406020024, F.Cu at (107.4, 62.3)
- added U1: STM32WB55CEUx, Package_DFN_QFN:QFN-48-1EP_7x7mm_P0.5mm_EP5.6x5.6mm, F.Cu at (112.0, 72.2)
- added U2: USBLC6-2SC6, Package_TO_SOT_SMD:SOT-23-6, F.Cu at (114.8, 59.4)
- added U3: MIC5365-3.3YD5, Package_TO_SOT_SMD:TSOT-23-5, F.Cu at (114.8, 64.0)
- added Y1: Crystal_GND24, Crystal:Crystal_SMD_2016-4Pin_2.0x1.6mm, F.Cu at (97.9, 87.2)
- added Y2: 32kHz768, Crystal:Crystal_SMD_3215-2Pin_3.2x1.5mm, F.Cu at (98.4, 83.7)
