File: VCAT/Kevin/kevin.kicad_sch (KiCad schematic)
At the start: 0 parts

Commit message: meow
Parts:
- added C1, C10, C14, C2, C3: 4.7u, Capacitor_SMD:C_0603_1608Metric, symbol Device:C
- added C11, C12, C13, C19, C4, C5, C6, C7, C8, C9: 100n, Capacitor_SMD:C_0402_1005Metric, symbol Device:C
- added C15, C16: 10p, Capacitor_SMD:C_0402_1005Metric, symbol Device:C
- added C17: .8p, Capacitor_SMD:C_0402_1005Metric, symbol Device:C
- added C18: .3p, Capacitor_SMD:C_0402_1005Metric, symbol Device:C
- added D1: LED, LED_SMD:LED_0402_1005Metric, symbol Device:LED
- added FLT1: DLF162500LT-5028A1, Starter Footprint:DLF162500LT-5028A1, symbol Starter Library:DLF162500LT-5028A1
- added J1: USB_C_Receptacle_USB2.0_16P, Connector_USB:USB_C_Receptacle_GCT_USB4105-xx-A_16P_TopMnt_Horizontal, symbol Connector:USB_C_Receptacle_USB2.0_16P
- added J2: Conn_ARM_SWD_TagConnect_TC2030, Connector_Molex:Molex_PicoBlade_53048-0410_1x04_P1.25mm_Horizontal, symbol Connector:Conn_ARM_SWD_TagConnect_TC2030
- added J3: Conn_01x04, Package_TO_SOT_SMD:TSOT-23-5, symbol Connector_Generic:Conn_01x04
- added J4: Conn_Coaxial, Connector:Tag-Connect_TC2030-IDC-FP_2x03_P1.27mm_Vertical, symbol Connector:Conn_Coaxial
- added L1: 10n, Inductor_SMD:L_0402_1005Metric, symbol Device:L
- added L2: 10u, Inductor_SMD:L_0805_2012Metric, symbol Device:L
- added L3: 2.7n, Inductor_SMD:L_0402_1005Metric, symbol Device:L
- added R1, R2, R6: 5.1k, Resistor_SMD:R_0402_1005Metric, symbol Device:R
- added R3, R4, R5, R7: 220R, Resistor_SMD:R_0402_1005Metric, symbol Device:R
- added SW1: SW_Push, Button_Switch_THT:SW_NKK_GW12LJP, symbol Switch:SW_Push
- added U1: MIC5365-3.3YD5, Button_Switch_SMD:SW_SPST_CK_RS282G05A3, symbol Regulator_Linear:MIC5365-3.3YD5
- added U2: USBLC6-2SC6, Package_TO_SOT_SMD:SOT-23-6, symbol Power_Protection:USBLC6-2SC6
- added U3: STM32WB55CEU6, Package_DFN_QFN:QFN-48-1EP_7x7mm_P0.5mm_EP5.6x5.6mm, symbol MCU_ST_STM32WB:STM32WB55CEUx
- added X1: 32.768kHz, Crystal:Crystal_SMD_2012-2Pin_2.0x1.2mm, symbol Device:Crystal
- added X2: 32mHz, Connector_Coaxial:U.FL_Hirose_U.FL-R-SMT-1_Vertical, symbol Device:Crystal_GND24
Connections:
- new net: R7.2, SW1.1
- new net: C15.1, U3.3 (PC15), X1.1
- new net: C16.1, U3.2 (PC14), X1.2
- new net: L1.1, U3.33 (VLXSMPS)
- new net: L1.2, L2.1
- new net +3.3V: C10.1, C11.1, C12.1, C2.1, C3.1, C4.1, C5.1, C6.1, C7.1, C8.1, C9.1, J2.1 (VCC), J3.4 (Pin_4), SW1.2, U1.5 (VOUT), U3.1 (VBAT), U3.20 (VDD), U3.23 (VDDRF), U3.34 (VDDSMPS), U3.35 (VDD), U3.40 (VDDUSB), U3.48 (VDD)
- new net +5V: C1.1, J1.A4 (VBUS), J1.A9 (VBUS), J1.B4 (VBUS), J1.B9 (VBUS), U1.1 (VIN), U1.3 (EN), U2.5 (VBUS)
- new net BOOT0: C19.1, R6.1, R7.1, U3.4 (PH3)
- new net GND: C1.2, C10.2, C11.2, C12.2, C13.2, C14.2, C15.2, C16.2, C17.2, C18.2, C19.2, C2.2, C3.2, C4.2, C5.2, C6.2, C7.2, C8.2, C9.2, FLT1.2 (GND), FLT1.4 (GND), J1.A1 (GND), J1.A12 (GND), J1.B1 (GND), J1.B12 (GND), J1.SH (SHIELD), J2.5 (GND), J3.1 (Pin_1), J4.2 (Ext), R1.2, R2.2, R5.1, R6.2, U1.2 (GND), U2.2 (GND), U3.22 (VSSRF), U3.32 (VSSSMPS), U3.49 (VSS), X2.2 (G), X2.4 (G)
- new net HSE_IN: U3.25 (OSC_IN), X2.3
- new net HSE_OUT: U3.24 (OSC_OUT), X2.1
- new net LED_A: D1.2 (A), U3.16 (PA7)
- new net LED_K: D1.1 (K), R5.2
- new net RF: C17.1, L3.1, U3.21 (RF1)
- new net RF_ANT: FLT1.3 (OUT), J4.1 (In)
- new net RF_MATCH: C18.1, FLT1.1 (IN), L3.2
- new net SMPSFB: C14.1, L2.2, U3.31 (VFBSMPS)
- new net SWCLK4: J2.4 (SWCLK), U3.41 (PA14)
- new net SWDIO: J2.2 (SWDIO), U3.39 (PA13)
- new net SWD_NRST: C13.1, J2.3 (~{RESET}), U3.7 (NRST)
- new net SWO: J2.6 (SWO), U3.43 (PB3)
- new net UART_RX: R4.2, U3.12 (PA3)
- new net UART_RXC: J3.2 (Pin_2), R4.1
- new net UART_TX: R3.2, U3.11 (PA2)
- new net UART_TXC: J3.3 (Pin_3), R3.1
- new net USB_CC1: J1.A5 (CC1), R2.1
- new net USB_CC2: J1.B5 (CC2), R1.1
- new net USB_D+: J1.A6 (D+), J1.B6 (D+), U2.3 (I/O2), U2.4 (I/O2), U3.38 (PA12)
- new net USB_D-: J1.A7 (D-), J1.B7 (D-), U2.1 (I/O1), U2.6 (I/O1), U3.37 (PA11)
- no-connect marks 0 -> 22
Other:
- note added: "3(.3-1.8V)/220 ~ 7mA"
- note added: "The 5V to 3.3V Regulator"
- note added: "Week 1"
